Commit message: Reorganizing project structure

File: assets/robots/g1_29dof_mode_15_brainco_hand.urdf (robot description, URDF)
Before this commit: robot g1_29dof_mode_15_brainco_hand, 73 links, 72 joints
Links:
- removed link world
- link head_link: geometry collision mesh filename=../../meshes/head_link.STL; visual mesh filename=../../meshes/head_link.STL
- link left_ankle_pitch_link: geometry collision mesh filename=../../meshes/left_ankle_pitch_link.STL; visual mesh filename=../../meshes/left_ankle_pitch_link.STL
- link left_ankle_roll_link: geometry collision sphere radius=0.005; collision sphere radius=0.005
- link left_base2_link: geometry collision mesh filename=../../meshes/left_base2_link.STL; visual mesh filename=../../meshes/left_base2_link.STL
- link left_base_link: geometry collision mesh filename=../../meshes/left_base_link.STL; visual mesh filename=../../meshes/left_base_link.STL
- link left_elbow_link: geometry collision mesh filename=../../meshes/left_elbow_link.STL; visual mesh filename=../../meshes/left_elbow_link.STL
- link left_hip_pitch_link: geometry collision mesh filename=../../meshes/left_hip_pitch_link.STL; visual mesh filename=../../meshes/left_hip_pitch_link.STL
- link left_hip_roll_link: geometry collision mesh filename=../../meshes/left_hip_roll_link.STL; visual mesh filename=../../meshes/left_hip_roll_link.STL
- link left_hip_yaw_link: geometry collision mesh filename=../../meshes/left_hip_yaw_link.STL; visual mesh filename=../../meshes/left_hip_yaw_link.STL
- link left_index_distal_Link: geometry collision mesh filename=../../meshes/left_index_distal_Link.STL; visual mesh filename=../../meshes/left_index_distal_Link.STL
- link left_index_proximal_Link: geometry collision mesh filename=../../meshes/left_index_proximal_Link.STL; visual mesh filename=../../meshes/left_index_proximal_Link.STL
- link left_index_tip_Link: geometry collision mesh filename=../../meshes/left_index_tip_Link.STL; visual mesh filename=../../meshes/left_index_tip_Link.STL
- link left_knee_link: geometry collision mesh filename=../../meshes/left_knee_link.STL; visual mesh filename=../../meshes/left_knee_link.STL
- link left_middle_distal_Link: geometry collision mesh filename=../../meshes/left_middle_distal_Link.STL; visual mesh filename=../../meshes/left_middle_distal_Link.STL
- link left_middle_proximal_Link: geometry collision mesh filename=../../meshes/left_middle_proximal_Link.STL; visual mesh filename=../../meshes/left_middle_proximal_Link.STL
- link left_middle_tip_Link: geometry collision mesh filename=../../meshes/left_middle_tip_Link.STL; visual mesh filename=../../meshes/left_middle_tip_Link.STL
- link left_pinky_distal_Link: geometry collision mesh filename=../../meshes/left_pinky_distal_Link.STL; visual mesh filename=../../meshes/left_pinky_distal_Link.STL
- link left_pinky_proximal_Link: geometry collision mesh filename=../../meshes/left_pinky_proximal_Link.STL; visual mesh filename=../../meshes/left_pinky_proximal_Link.STL
- link left_pinky_tip_Link: geometry collision mesh filename=../../meshes/left_pinky_tip_Link.STL; visual mesh filename=../../meshes/left_pinky_tip_Link.STL
- link left_ring_distal_Link: geometry collision mesh filename=../../meshes/left_ring_distal_Link.STL; visual mesh filename=../../meshes/left_ring_distal_Link.STL
- link left_ring_proximal_Link: geometry collision mesh filename=../../meshes/left_ring_proximal_Link.STL; visual mesh filename=../../meshes/left_ring_proximal_Link.STL
- link left_ring_tip_Link: geometry collision mesh filename=../../meshes/left_ring_tip_Link.STL; visual mesh filename=../../meshes/left_ring_tip_Link.STL
- link left_shoulder_pitch_link: geometry collision cylinder length=0.05 radius=0.03; visual mesh filename=../../meshes/left_shoulder_pitch_link.STL
- link left_shoulder_roll_link: geometry collision cylinder length=0.03 radius=0.03; visual mesh filename=../../meshes/left_shoulder_roll_link.STL
- link left_shoulder_yaw_link: geometry collision mesh filename=../../meshes/left_shoulder_yaw_link.STL; visual mesh filename=../../meshes/left_shoulder_yaw_link.STL
- link left_thumb_distal_Link: geometry collision mesh filename=../../meshes/left_thumb_distal_Link.STL; visual mesh filename=../../meshes/left_thumb_distal_Link.STL
- link left_thumb_metacarpal_Link: geometry collision mesh filename=../../meshes/left_thumb_metacarpal_Link.STL; visual mesh filename=../../meshes/left_thumb_metacarpal_Link.STL
- link left_thumb_proximal_Link: geometry collision mesh filename=../../meshes/left_thumb_proximal_Link.STL; visual mesh filename=../../meshes/left_thumb_proximal_Link.STL
- link left_thumb_tip_Link: geometry collision mesh filename=../../meshes/left_thumb_tip_Link.STL; visual mesh filename=../../meshes/left_thumb_tip_Link.STL
- link left_wrist_pitch_link: geometry collision mesh filename=../../meshes/left_wrist_pitch_link.STL; visual mesh filename=../../meshes/left_wrist_pitch_link.STL
- link left_wrist_roll_link: geometry collision mesh filename=../../meshes/left_wrist_roll_link.STL; visual mesh filename=../../meshes/left_wrist_roll_link.STL
- link left_wrist_yaw_link: geometry collision mesh filename=../../meshes/left_wrist_yaw_link.STL; visual mesh filename=../../meshes/left_wrist_yaw_link.STL
- link logo_link: geometry collision mesh filename=../../meshes/logo_link.STL; visual mesh filename=../../meshes/logo_link.STL
- link pelvis: geometry visual mesh filename=../../meshes/pelvis_ver0529.STL
- link right_ankle_pitch_link: geometry collision mesh filename=../../meshes/right_ankle_pitch_link.STL; visual mesh filename=../../meshes/right_ankle_pitch_link.STL
- link right_ankle_roll_link: geometry collision sphere radius=0.005; collision sphere radius=0.005
- link right_base2_link: geometry collision mesh filename=../../meshes/right_base2_link.STL; visual mesh filename=../../meshes/right_base2_link.STL
- link right_base_link: geometry collision mesh filename=../../meshes/right_base_link.STL; visual mesh filename=../../meshes/right_base_link.STL
- link right_elbow_link: geometry collision mesh filename=../../meshes/right_elbow_link.STL; visual mesh filename=../../meshes/right_elbow_link.STL
- link right_hip_pitch_link: geometry collision mesh filename=../../meshes/right_hip_pitch_link.STL; visual mesh filename=../../meshes/right_hip_pitch_link.STL
- link right_hip_roll_link: geometry collision mesh filename=../../meshes/right_hip_roll_link.STL; visual mesh filename=../../meshes/right_hip_roll_link.STL
- link right_hip_yaw_link: geometry collision mesh filename=../../meshes/right_hip_yaw_link.STL; visual mesh filename=../../meshes/right_hip_yaw_link.STL
- link right_index_distal_link: geometry collision mesh filename=../../meshes/right_index_distal_link.STL; visual mesh filename=../../meshes/right_index_distal_link.STL
- link right_index_proximal_link: geometry collision mesh filename=../../meshes/right_index_proximal_link.STL; visual mesh filename=../../meshes/right_index_proximal_link.STL
- link right_index_tip: geometry collision mesh filename=../../meshes/right_index_tip.STL; visual mesh filename=../../meshes/right_index_tip.STL
- link right_knee_link: geometry collision mesh filename=../../meshes/right_knee_link.STL; visual mesh filename=../../meshes/right_knee_link.STL
- link right_middle_distal_link: geometry collision mesh filename=../../meshes/right_middle_distal_link.STL; visual mesh filename=../../meshes/right_middle_distal_link.STL
- link right_middle_proximal_link: geometry collision mesh filename=../../meshes/right_middle_proximal_link.STL; visual mesh filename=../../meshes/right_middle_proximal_link.STL
- link right_middle_tip: geometry collision mesh filename=../../meshes/right_middle_tip.STL; visual mesh filename=../../meshes/right_middle_tip.STL
- link right_pinky_distal_link: geometry collision mesh filename=../../meshes/right_pinky_distal_link.STL; visual mesh filename=../../meshes/right_pinky_distal_link.STL
- link right_pinky_proximal_link: geometry collision mesh filename=../../meshes/right_pinky_proximal_link.STL; visual mesh filename=../../meshes/right_pinky_proximal_link.STL
- link right_pinky_tip: geometry collision mesh filename=../../meshes/right_pinky_tip.STL; visual mesh filename=../../meshes/right_pinky_tip.STL
- link right_ring_distal_link: geometry collision mesh filename=../../meshes/right_ring_distal_link.STL; visual mesh filename=../../meshes/right_ring_distal_link.STL
- link right_ring_proximal_link: geometry collision mesh filename=../../meshes/right_ring_proximal_link.STL; visual mesh filename=../../meshes/right_ring_proximal_link.STL
- link right_ring_tip: geometry collision mesh filename=../../meshes/right_ring_tip.STL; visual mesh filename=../../meshes/right_ring_tip.STL
- link right_shoulder_pitch_link: geometry collision cylinder length=0.05 radius=0.03; visual mesh filename=../../meshes/right_shoulder_pitch_link.STL
- link right_shoulder_roll_link: geometry collision cylinder length=0.03 radius=0.03; visual mesh filename=../../meshes/right_shoulder_roll_link.STL
- link right_shoulder_yaw_link: geometry collision mesh filename=../../meshes/right_shoulder_yaw_link.STL; visual mesh filename=../../meshes/right_shoulder_yaw_link.STL
- link right_thumb_distal_link: geometry collision mesh filename=../../meshes/right_thumb_distal_link.STL; visual mesh filename=../../meshes/right_thumb_distal_link.STL
- link right_thumb_metacarpal_link: geometry collision mesh filename=../../meshes/right_thumb_metacarpal_link.STL; visual mesh filename=../../meshes/right_thumb_metacarpal_link.STL
- link right_thumb_proximal_link: geometry collision mesh filename=../../meshes/right_thumb_proximal_link.STL; visual mesh filename=../../meshes/right_thumb_proximal_link.STL
- link right_thumb_tip: geometry collision mesh filename=../../meshes/right_thumb_tip.STL; visual mesh filename=../../meshes/right_thumb_tip.STL
- link right_wrist_pitch_link: geometry collision mesh filename=../../meshes/right_wrist_pitch_link.STL; visual mesh filename=../../meshes/right_wrist_pitch_link.STL
- link right_wrist_roll_link: geometry collision mesh filename=../../meshes/right_wrist_roll_link.STL; visual mesh filename=../../meshes/right_wrist_roll_link.STL
- link right_wrist_yaw_link: geometry collision mesh filename=../../meshes/right_wrist_yaw_link.STL; visual mesh filename=../../meshes/right_wrist_yaw_link.STL
- link torso_link: geometry collision mesh filename=../../meshes/torso_link_rev_1_0.STL; visual mesh filename=../../meshes/torso_link_rev_1_0.STL
- link waist_roll_link: geometry visual mesh filename=../../meshes/waist_roll_link_rev_1_0.STL
- link waist_yaw_link: geometry visual mesh filename=../../meshes/waist_yaw_link_rev_1_0.STL
Joints:
- removed joint floating_base_joint

File: assets/robots/g1_fixed.urdf (robot description, URDF)
Before this commit: robot g1_29dof_mode_15_brainco_hand, 72 links, 71 joints
Links:
- link head_link: geometry collision mesh filename=../../meshes/head_link.STL; visual mesh filename=../../meshes/head_link.STL
- link left_ankle_pitch_link: geometry collision mesh filename=../../meshes/left_ankle_pitch_link.STL; visual mesh filename=../../meshes/left_ankle_pitch_link.STL
- link left_ankle_roll_link: geometry collision sphere radius=0.005; collision sphere radius=0.005
- link left_base2_link: geometry collision mesh filename=../../meshes/left_base2_link.STL; visual mesh filename=../../meshes/left_base2_link.STL
- link left_base_link: geometry collision mesh filename=../../meshes/left_base_link.STL; visual mesh filename=../../meshes/left_base_link.STL
- link left_elbow_link: geometry collision mesh filename=../../meshes/left_elbow_link.STL; visual mesh filename=../../meshes/left_elbow_link.STL
- link left_hip_pitch_link: geometry collision mesh filename=../../meshes/left_hip_pitch_link.STL; visual mesh filename=../../meshes/left_hip_pitch_link.STL
- link left_hip_roll_link: geometry collision mesh filename=../../meshes/left_hip_roll_link.STL; visual mesh filename=../../meshes/left_hip_roll_link.STL
- link left_hip_yaw_link: geometry collision mesh filename=../../meshes/left_hip_yaw_link.STL; visual mesh filename=../../meshes/left_hip_yaw_link.STL
- link left_index_distal_Link: geometry collision mesh filename=../../meshes/left_index_distal_Link.STL; visual mesh filename=../../meshes/left_index_distal_Link.STL
- link left_index_proximal_Link: geometry collision mesh filename=../../meshes/left_index_proximal_Link.STL; visual mesh filename=../../meshes/left_index_proximal_Link.STL
- link left_index_tip_Link: geometry collision mesh filename=../../meshes/left_index_tip_Link.STL; visual mesh filename=../../meshes/left_index_tip_Link.STL
- link left_knee_link: geometry collision mesh filename=../../meshes/left_knee_link.STL; visual mesh filename=../../meshes/left_knee_link.STL
- link left_middle_distal_Link: geometry collision mesh filename=../../meshes/left_middle_distal_Link.STL; visual mesh filename=../../meshes/left_middle_distal_Link.STL
- link left_middle_proximal_Link: geometry collision mesh filename=../../meshes/left_middle_proximal_Link.STL; visual mesh filename=../../meshes/left_middle_proximal_Link.STL
- link left_middle_tip_Link: geometry collision mesh filename=../../meshes/left_middle_tip_Link.STL; visual mesh filename=../../meshes/left_middle_tip_Link.STL
- link left_pinky_distal_Link: geometry collision mesh filename=../../meshes/left_pinky_distal_Link.STL; visual mesh filename=../../meshes/left_pinky_distal_Link.STL
- link left_pinky_proximal_Link: geometry collision mesh filename=../../meshes/left_pinky_proximal_Link.STL; visual mesh filename=../../meshes/left_pinky_proximal_Link.STL
- link left_pinky_tip_Link: geometry collision mesh filename=../../meshes/left_pinky_tip_Link.STL; visual mesh filename=../../meshes/left_pinky_tip_Link.STL
- link left_ring_distal_Link: geometry collision mesh filename=../../meshes/left_ring_distal_Link.STL; visual mesh filename=../../meshes/left_ring_distal_Link.STL
- link left_ring_proximal_Link: geometry collision mesh filename=../../meshes/left_ring_proximal_Link.STL; visual mesh filename=../../meshes/left_ring_proximal_Link.STL
- link left_ring_tip_Link: geometry collision mesh filename=../../meshes/left_ring_tip_Link.STL; visual mesh filename=../../meshes/left_ring_tip_Link.STL
- link left_shoulder_pitch_link: geometry collision cylinder length=0.05 radius=0.03; visual mesh filename=../../meshes/left_shoulder_pitch_link.STL
- link left_shoulder_roll_link: geometry collision cylinder length=0.03 radius=0.03; visual mesh filename=../../meshes/left_shoulder_roll_link.STL
- link left_shoulder_yaw_link: geometry collision mesh filename=../../meshes/left_shoulder_yaw_link.STL; visual mesh filename=../../meshes/left_shoulder_yaw_link.STL
- link left_thumb_distal_Link: geometry collision mesh filename=../../meshes/left_thumb_distal_Link.STL; visual mesh filename=../../meshes/left_thumb_distal_Link.STL
- link left_thumb_metacarpal_Link: geometry collision mesh filename=../../meshes/left_thumb_metacarpal_Link.STL; visual mesh filename=../../meshes/left_thumb_metacarpal_Link.STL
- link left_thumb_proximal_Link: geometry collision mesh filename=../../meshes/left_thumb_proximal_Link.STL; visual mesh filename=../../meshes/left_thumb_proximal_Link.STL
- link left_thumb_tip_Link: geometry collision mesh filename=../../meshes/left_thumb_tip_Link.STL; visual mesh filename=../../meshes/left_thumb_tip_Link.STL
- link left_wrist_pitch_link: geometry collision mesh filename=../../meshes/left_wrist_pitch_link.STL; visual mesh filename=../../meshes/left_wrist_pitch_link.STL
- link left_wrist_roll_link: geometry collision mesh filename=../../meshes/left_wrist_roll_link.STL; visual mesh filename=../../meshes/left_wrist_roll_link.STL
- link left_wrist_yaw_link: geometry collision mesh filename=../../meshes/left_wrist_yaw_link.STL; visual mesh filename=../../meshes/left_wrist_yaw_link.STL
- link logo_link: geometry collision mesh filename=../../meshes/logo_link.STL; visual mesh filename=../../meshes/logo_link.STL
- link pelvis: geometry visual mesh filename=../../meshes/pelvis_ver0529.STL
- link right_ankle_pitch_link: geometry collision mesh filename=../../meshes/right_ankle_pitch_link.STL; visual mesh filename=../../meshes/right_ankle_pitch_link.STL
- link right_ankle_roll_link: geometry collision sphere radius=0.005; collision sphere radius=0.005
- link right_base2_link: geometry collision mesh filename=../../meshes/right_base2_link.STL; visual mesh filename=../../meshes/right_base2_link.STL
- link right_base_link: geometry collision mesh filename=../../meshes/right_base_link.STL; visual mesh filename=../../meshes/right_base_link.STL
- link right_elbow_link: geometry collision mesh filename=../../meshes/right_elbow_link.STL; visual mesh filename=../../meshes/right_elbow_link.STL
- link right_hip_pitch_link: geometry collision mesh filename=../../meshes/right_hip_pitch_link.STL; visual mesh filename=../../meshes/right_hip_pitch_link.STL
- link right_hip_roll_link: geometry collision mesh filename=../../meshes/right_hip_roll_link.STL; visual mesh filename=../../meshes/right_hip_roll_link.STL
- link right_hip_yaw_link: geometry collision mesh filename=../../meshes/right_hip_yaw_link.STL; visual mesh filename=../../meshes/right_hip_yaw_link.STL
- link right_index_distal_link: geometry collision mesh filename=../../meshes/right_index_distal_link.STL; visual mesh filename=../../meshes/right_index_distal_link.STL
- link right_index_proximal_link: geometry collision mesh filename=../../meshes/right_index_proximal_link.STL; visual mesh filename=../../meshes/right_index_proximal_link.STL
- link right_index_tip: geometry collision mesh filename=../../meshes/right_index_tip.STL; visual mesh filename=../../meshes/right_index_tip.STL
- link right_knee_link: geometry collision mesh filename=../../meshes/right_knee_link.STL; visual mesh filename=../../meshes/right_knee_link.STL
- link right_middle_distal_link: geometry collision mesh filename=../../meshes/right_middle_distal_link.STL; visual mesh filename=../../meshes/right_middle_distal_link.STL
- link right_middle_proximal_link: geometry collision mesh filename=../../meshes/right_middle_proximal_link.STL; visual mesh filename=../../meshes/right_middle_proximal_link.STL
- link right_middle_tip: geometry collision mesh filename=../../meshes/right_middle_tip.STL; visual mesh filename=../../meshes/right_middle_tip.STL
- link right_pinky_distal_link: geometry collision mesh filename=../../meshes/right_pinky_distal_link.STL; visual mesh filename=../../meshes/right_pinky_distal_link.STL
- link right_pinky_proximal_link: geometry collision mesh filename=../../meshes/right_pinky_proximal_link.STL; visual mesh filename=../../meshes/right_pinky_proximal_link.STL
- link right_pinky_tip: geometry collision mesh filename=../../meshes/right_pinky_tip.STL; visual mesh filename=../../meshes/right_pinky_tip.STL
- link right_ring_distal_link: geometry collision mesh filename=../../meshes/right_ring_distal_link.STL; visual mesh filename=../../meshes/right_ring_distal_link.STL
- link right_ring_proximal_link: geometry collision mesh filename=../../meshes/right_ring_proximal_link.STL; visual mesh filename=../../meshes/right_ring_proximal_link.STL
- link right_ring_tip: geometry collision mesh filename=../../meshes/right_ring_tip.STL; visual mesh filename=../../meshes/right_ring_tip.STL
- link right_shoulder_pitch_link: geometry collision cylinder length=0.05 radius=0.03; visual mesh filename=../../meshes/right_shoulder_pitch_link.STL
- link right_shoulder_roll_link: geometry collision cylinder length=0.03 radius=0.03; visual mesh filename=../../meshes/right_shoulder_roll_link.STL
- link right_shoulder_yaw_link: geometry collision mesh filename=../../meshes/right_shoulder_yaw_link.STL; visual mesh filename=../../meshes/right_shoulder_yaw_link.STL
- link right_thumb_distal_link: geometry collision mesh filename=../../meshes/right_thumb_distal_link.STL; visual mesh filename=../../meshes/right_thumb_distal_link.STL
- link right_thumb_metacarpal_link: geometry collision mesh filename=../../meshes/right_thumb_metacarpal_link.STL; visual mesh filename=../../meshes/right_thumb_metacarpal_link.STL
- link right_thumb_proximal_link: geometry collision mesh filename=../../meshes/right_thumb_proximal_link.STL; visual mesh filename=../../meshes/right_thumb_proximal_link.STL
- link right_thumb_tip: geometry collision mesh filename=../../meshes/right_thumb_tip.STL; visual mesh filename=../../meshes/right_thumb_tip.STL
- link right_wrist_pitch_link: geometry collision mesh filename=../../meshes/right_wrist_pitch_link.STL; visual mesh filename=../../meshes/right_wrist_pitch_link.STL
- link right_wrist_roll_link: geometry collision mesh filename=../../meshes/right_wrist_roll_link.STL; visual mesh filename=../../meshes/right_wrist_roll_link.STL
- link right_wrist_yaw_link: geometry collision mesh filename=../../meshes/right_wrist_yaw_link.STL; visual mesh filename=../../meshes/right_wrist_yaw_link.STL
- link torso_link: geometry collision mesh filename=../../meshes/torso_link_rev_1_0.STL; visual mesh filename=../../meshes/torso_link_rev_1_0.STL
- link waist_roll_link: geometry visual mesh filename=../../meshes/waist_roll_link_rev_1_0.STL
- link waist_yaw_link: geometry visual mesh filename=../../meshes/waist_yaw_link_rev_1_0.STL
